File: hardware/HMC6343 Breakout.sch (EAGLE design)
At the start: 15 parts, among them U1 HMC6343A

Commit message: v10, ready for reds
Other:
- note added: "v10"
- note removed: "v01"
Changed lines of the file:
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@@
 <plain>
 <text x="152.4" y="7.62" size="2.54" layer="94">Jordan McConnell</text>
-<text x="238.76" y="7.62" size="2.54" layer="94">v01</text>
+<text x="238.76" y="7.62" size="2.54" layer="94">v10</text>
 <text x="137.16" y="81.28" size="1.778" layer="97">I2C Address: 0x32</text>
 </plain>
